Commit message: Added hummingbird.xacro

File: mav_description/urdf/multirotor_base.xacro (robot description, xacro)
@@ -36,5 +36,5 @@
     Macro for the multirotor's body/base
   -->
-  <xacro:macro name="multirotor_base_xacro"
+  <xacro:macro name="multirotor_base"
     params="robot_namespace mass length width heigth mesh_file *inertia">
     <link name="${robot_namespace}/base_link">
@@ -65,3 +65,26 @@
     </joint>
   </xacro:macro>
+  <!--
+    Macro for the multirotor's vertical rotor
+  -->
+  <xacro:macro name="vertical_rotor"
+    params="robot_namespace suffix direction parent mass radius id color *origin *inertia">
+    <link name="${robot_namespace}/rotor_${id}">
+      <inertial>
+        <mass value="${mass}"/> <!-- [kg] -->
+        <xacro:insert_block name="inertia"/>
+      </inertial>
+      <visual>
+        <geometry>
+          <mesh filename="package://mav_description/meshes/propeller_${direction}.dae"
+            scale="${radius} ${radius} ${radius}"/> <!-- [m] [m] [m] -->
+        </geometry>
+      </visual>
+      <collision>
+        <geometry>
+          <cylinder length="0.005" radius="${radius}"/> <!-- [m] -->
+        </geometry>
+      </collision>
+    </link>
+  </xacro:macro>
 </robot>

Commit message: Added hummingbird_base.xacro

File: mav_description/urdf/multirotor_base.xacro (robot description, xacro)
@@ -21,5 +21,5 @@
     <inertia ixx="${(1.0/12.0) * mass * (y*y + z*z)}" ixy="0.0" ixz="0.0"
              iyy="${(1.0/12.0) * mass * (x*x + z*z)}" iyz="0.0"
-             izz="${(1.0/12.0) * mass * (x*x + y*y)}"/>
+             izz="${(1.0/12.0) * mass * (x*x + y*y)}"/> <!-- [kg m^2] ... -->
   </xacro:macro>
   <!--
@@ -61,5 +61,5 @@
     <joint name="${robot_namespace}/base_joint" type="fixed">
       <origin xyz="0 0 0" rpy="0 0 0"/>
-      <parent link="${robot_namespace}/baselink"/>
+      <parent link="${robot_namespace}/base_link"/>
       <child link="${robot_namespace}/base_link_inertia"/>
     </joint>
