Commit message: Updated multirotor_base.xacro

File: mav_description/urdf/hummingbird.xacro (robot description, xacro)
@@ -13,8 +13,8 @@
   limitations under the License.
 -->
-<robot xmlns:xacro="http://ros.org/wiki/xacro">
+<robot name="hummingbird" xmlns:xacro="http://ros.org/wiki/xacro">
   <!--
     Include the hummingbird base xacro
   -->
-  <xacro:include filename="$(find mav_description)/urdf/hummingbird_base.xacro"/>
+  <xacro:include filename="$(find-pkg-share mav_description)/urdf/hummingbird_base.xacro"/>
 </robot>

File: mav_description/urdf/hummingbird_base.xacro (robot description, xacro)
@@ -25,5 +25,5 @@
   <xacro:property name="body_height" value="0.12"/> <!-- [m] -->
   <xacro:property name="rotor_mass" value="0.009"/> <!-- [kg] -->
-  <xacro:property name="rotor_radius" value="0.1"> <!-- [m] -->
+  <xacro:property name="rotor_radius" value="0.1"/> <!-- [m] -->
   <xacro:property name="arm_length" value="0.17"/> <!-- [m] -->
   <xacro:property name="robot_z_offset" value="0.01"/> <!-- [m]-->
@@ -46,5 +46,5 @@
     Include the multirotor base xacro
   -->
-  <xacro:include filename="$(find mav_description)/urdf/multirotor_base.xacro"/>
+  <xacro:include filename="$(find-pkg-share mav_description)/urdf/multirotor_base.xacro"/>
   <!--
     Instantiate the multirotor_base macro

File: mav_description/urdf/multirotor_base.xacro (robot description, xacro)
@@ -87,4 +87,10 @@
       </collision>
     </link>
+    <joint name="${robot_namespace}/robot_${id}_joint" type="continuous">
+      <xacro:insert_block name="origin"/>
+      <axis xyz="0 0 1"/>
+      <parent link="${parent}"/>
+      <child link="${robot_namespace}/robot_${id}"/>
+    </joint>
   </xacro:macro>
 </robot>

Commit message: Update hummingbird.xacro

File: mav_description/urdf/hummingbird.xacro (robot description, xacro)
@@ -17,4 +17,4 @@
     Include the hummingbird base xacro
   -->
-  <xacro:include filename="$(find-pkg-share mav_description)/urdf/hummingbird_base.xacro"/>
+  <xacro:include filename="$(find mav_description)/urdf/hummingbird_base.xacro"/>
 </robot>

File: mav_description/urdf/hummingbird_base.xacro (robot description, xacro)
@@ -29,4 +29,8 @@
   <xacro:property name="robot_z_offset" value="0.01"/> <!-- [m]-->
   <!--
+    Include the multirotor base xacro
+  -->
+  <xacro:include filename="$(find mav_description)/urdf/multirotor_base.xacro"/>
+  <!--
     Property for the body's inertia
   -->
@@ -42,9 +46,5 @@
     <xacro:box_inertia x="${rotor_radius}" y="0.015" z="0.003"
       mass="${rotor_mass}"/>
-  </xacro:property/>
-  <!--
-    Include the multirotor base xacro
-  -->
-  <xacro:include filename="$(find-pkg-share mav_description)/urdf/multirotor_base.xacro"/>
+  </xacro:property>
   <!--
     Instantiate the multirotor_base macro
