Commit message: Update multirobot_base.xacro for propeller color

File: mav_description/urdf/multirotor_base.urdf.xacro (robot description, xacro)
@@ -93,4 +93,7 @@
       <child link="${robot_namespace}/rotor_${id}"/>
     </joint>
+    <gazebo reference="${robot_namespace}/rotor_${id}">
+      <material>Gazebo/${color}</material>
+    </gazebo>
   </xacro:macro>
 </robot>
