Commit message: Update hummingbird.urdf.xacro

File: mav_description/urdf/hummingbird_base.urdf.xacro (robot description, xacro)
@@ -69,5 +69,5 @@
   <xacro:vertical_rotor robot_namespace="${namespace}" suffix="left"
     direction="ccw" parent="${namespace}/base_link" mass="${rotor_mass}"
-    radius="${rotor_radius}" id="0" color="Blue">
+    radius="${rotor_radius}" id="1" color="Blue">
     <origin xyz="0 ${arm_length} ${robot_z_offset}" rpy="0 0 0"/>
     <xacro:insert_block name="robot_inertia"/>
@@ -78,5 +78,5 @@
   <xacro:vertical_rotor robot_namespace="${namespace}" suffix="back"
     direction="cw" parent="${namespace}/base_link" mass="${rotor_mass}"
-    radius="${rotor_radius}" id="0" color="Blue">
+    radius="${rotor_radius}" id="2" color="Blue">
     <origin xyz="-${arm_length} 0 ${robot_z_offset}" rpy="0 0 0"/>
     <xacro:insert_block name="robot_inertia"/>
@@ -87,5 +87,5 @@
   <xacro:vertical_rotor robot_namespace="${namespace}" suffix="right"
     direction="ccw" parent="${namespace}/base_link" mass="${rotor_mass}"
-    radius="${rotor_radius}" id="0" color="Blue">
+    radius="${rotor_radius}" id="3" color="Blue">
     <origin xyz="0 -${arm_length} ${robot_z_offset}" rpy="0 0 0"/>
     <xacro:insert_block name="robot_inertia"/>

File: mav_description/urdf/multirotor_base.urdf.xacro (robot description, xacro)
@@ -87,9 +87,9 @@
       </collision>
     </link>
-    <joint name="${robot_namespace}/robot_${id}_joint" type="continuous">
+    <joint name="${robot_namespace}/rotor_${id}_joint" type="continuous">
       <xacro:insert_block name="origin"/>
       <axis xyz="0 0 1"/>
       <parent link="${parent}"/>
-      <child link="${robot_namespace}/robot_${id}"/>
+      <child link="${robot_namespace}/rotor_${id}"/>
     </joint>
   </xacro:macro>

Commit message: Update *.urdf.xacro for bug fix of *.dae include

File: mav_description/urdf/hummingbird_base.urdf.xacro (robot description, xacro)
@@ -19,5 +19,5 @@
   -->
   <xacro:property name="namespace" value="$(arg namespace)"/>
-  <xacro:property name="mav_mesh_file" value="package://mav_description/meshes/hummingbird.dae"/>
+  <xacro:property name="mav_mesh_file" value="file://$(find mav_description)/meshes/hummingbird.dae"/>
   <xacro:property name="body_mass" value="0.68"/> <!-- [kg] -->
   <xacro:property name="body_length" value="0.1"/> <!-- [m] -->

File: mav_description/urdf/multirotor_base.urdf.xacro (robot description, xacro)
@@ -77,5 +77,5 @@
       <visual>
         <geometry>
-          <mesh filename="package://mav_description/meshes/propeller_${direction}.dae"
+          <mesh filename="file://$(find mav_description)/meshes/propeller_${direction}.dae"
             scale="${radius} ${radius} ${radius}"/> <!-- [m] [m] [m] -->
         </geometry>

Commit message: Update hummingbird_base.xacro

File: mav_description/urdf/hummingbird_base.urdf.xacro (robot description, xacro)
@@ -27,5 +27,5 @@
   <xacro:property name="rotor_radius" value="0.1"/> <!-- [m] -->
   <xacro:property name="arm_length" value="0.17"/> <!-- [m] -->
-  <xacro:property name="robot_z_offset" value="0.01"/> <!-- [m]-->
+  <xacro:property name="rotor_z_offset" value="0.01"/> <!-- [m]-->
   <!--
     Include the multirotor base xacro
@@ -41,7 +41,7 @@
   </xacro:property>
   <!--
-    Property for the single robot's inertia, assuming a cuboid shape
+    Property for the single rotor's inertia, assuming a cuboid shape
   -->
-  <xacro:property name="robot_inertia">
+  <xacro:property name="rotor_inertia">
     <xacro:box_inertia x="${rotor_radius}" y="0.015" z="0.003"
       mass="${rotor_mass}"/>
@@ -61,6 +61,6 @@
     direction="cw" parent="${namespace}/base_link" mass="${rotor_mass}"
     radius="${rotor_radius}" id="0" color="Red">
-    <origin xyz="${arm_length} 0 ${robot_z_offset}" rpy="0 0 0"/>
-    <xacro:insert_block name="robot_inertia"/>
+    <origin xyz="${arm_length} 0 ${rotor_z_offset}" rpy="0 0 0"/>
+    <xacro:insert_block name="rotor_inertia"/>
   </xacro:vertical_rotor>
   <!--
@@ -70,6 +70,6 @@
     direction="ccw" parent="${namespace}/base_link" mass="${rotor_mass}"
     radius="${rotor_radius}" id="1" color="Blue">
-    <origin xyz="0 ${arm_length} ${robot_z_offset}" rpy="0 0 0"/>
-    <xacro:insert_block name="robot_inertia"/>
+    <origin xyz="0 ${arm_length} ${rotor_z_offset}" rpy="0 0 0"/>
+    <xacro:insert_block name="rotor_inertia"/>
   </xacro:vertical_rotor>
   <!--
@@ -79,6 +79,6 @@
     direction="cw" parent="${namespace}/base_link" mass="${rotor_mass}"
     radius="${rotor_radius}" id="2" color="Blue">
-    <origin xyz="-${arm_length} 0 ${robot_z_offset}" rpy="0 0 0"/>
-    <xacro:insert_block name="robot_inertia"/>
+    <origin xyz="-${arm_length} 0 ${rotor_z_offset}" rpy="0 0 0"/>
+    <xacro:insert_block name="rotor_inertia"/>
   </xacro:vertical_rotor>
   <!--
@@ -88,6 +88,6 @@
     direction="ccw" parent="${namespace}/base_link" mass="${rotor_mass}"
     radius="${rotor_radius}" id="3" color="Blue">
-    <origin xyz="0 -${arm_length} ${robot_z_offset}" rpy="0 0 0"/>
-    <xacro:insert_block name="robot_inertia"/>
+    <origin xyz="0 -${arm_length} ${rotor_z_offset}" rpy="0 0 0"/>
+    <xacro:insert_block name="rotor_inertia"/>
   </xacro:vertical_rotor>
 </robot>
