Commit message: cleanup launch files

File: mav_description/urdf/hummingbird.urdf.xacro (robot description, xacro)
@@ -17,4 +17,4 @@
     Include the hummingbird base xacro
   -->
-  <xacro:include filename="$(find mav_description)/urdf/hummingbird_base.urdf.xacro"/>
+  <xacro:include filename="$(find mav_description)/urdf/hummingbird_base.urdf.xacro" />
 </robot>

File: mav_description/urdf/hummingbird_base.urdf.xacro (robot description, xacro)
@@ -18,18 +18,18 @@
     reference Novel Dynamic Inversion Architectur Design for Quadrocopter Control by Wang et al.
   -->
-  <xacro:property name="namespace" value="$(arg namespace)"/>
-  <xacro:property name="mav_mesh_file" value="file://$(find mav_description)/meshes/hummingbird.dae"/>
-  <xacro:property name="body_mass" value="0.68"/> <!-- [kg] -->
-  <xacro:property name="body_length" value="0.1"/> <!-- [m] -->
-  <xacro:property name="body_width" value="0.1"/> <!-- [m] -->
-  <xacro:property name="body_height" value="0.12"/> <!-- [m] -->
-  <xacro:property name="rotor_mass" value="0.009"/> <!-- [kg] -->
-  <xacro:property name="rotor_radius" value="0.1"/> <!-- [m] -->
-  <xacro:property name="arm_length" value="0.17"/> <!-- [m] -->
-  <xacro:property name="rotor_z_offset" value="0.01"/> <!-- [m]-->
+  <xacro:property name="namespace" value="$(arg namespace)" />
+  <xacro:property name="mav_mesh_file" value="file://$(find mav_description)/meshes/hummingbird.dae" />
+  <xacro:property name="body_mass" value="0.68" /> <!-- [kg] -->
+  <xacro:property name="body_length" value="0.1" /> <!-- [m] -->
+  <xacro:property name="body_width" value="0.1" /> <!-- [m] -->
+  <xacro:property name="body_height" value="0.12" /> <!-- [m] -->
+  <xacro:property name="rotor_mass" value="0.009" /> <!-- [kg] -->
+  <xacro:property name="rotor_radius" value="0.1" /> <!-- [m] -->
+  <xacro:property name="arm_length" value="0.17" /> <!-- [m] -->
+  <xacro:property name="rotor_z_offset" value="0.01" /> <!-- [m]-->
   <!--
     Include the multirotor base xacro
   -->
-  <xacro:include filename="$(find mav_description)/urdf/multirotor_base.urdf.xacro"/>
+  <xacro:include filename="$(find mav_description)/urdf/multirotor_base.urdf.xacro" />
   <!--
     Property for the body's inertia
@@ -38,5 +38,5 @@
     <inertia ixx="0.007" ixy="0.0" ixz="0.0"
              iyy="0.007" iyz="0.0"
-             izz="0.012"/> <!-- [kg m^2] ... -->
+             izz="0.012" /> <!-- [kg m^2] ... -->
   </xacro:property>
   <!--
@@ -45,5 +45,5 @@
   <xacro:property name="rotor_inertia">
     <xacro:box_inertia x="${rotor_radius}" y="0.015" z="0.003"
-      mass="${rotor_mass}"/>
+      mass="${rotor_mass}" />
   </xacro:property>
   <!--
@@ -53,5 +53,5 @@
     length="${body_length}" width="${body_width}" height="${body_height}"
     mesh_file="${mav_mesh_file}">
-    <xacro:insert_block name="body_inertia"/>
+    <xacro:insert_block name="body_inertia" />
   </xacro:multirotor_base>
   <!--
@@ -61,6 +61,6 @@
     direction="cw" parent="${namespace}/base_link" mass="${rotor_mass}"
     radius="${rotor_radius}" id="0" color="Red">
-    <origin xyz="${arm_length} 0 ${rotor_z_offset}" rpy="0 0 0"/>
-    <xacro:insert_block name="rotor_inertia"/>
+    <origin xyz="${arm_length} 0 ${rotor_z_offset}" rpy="0 0 0" />
+    <xacro:insert_block name="rotor_inertia" />
   </xacro:vertical_rotor>
   <!--
@@ -70,6 +70,6 @@
     direction="ccw" parent="${namespace}/base_link" mass="${rotor_mass}"
     radius="${rotor_radius}" id="1" color="Blue">
-    <origin xyz="0 ${arm_length} ${rotor_z_offset}" rpy="0 0 0"/>
-    <xacro:insert_block name="rotor_inertia"/>
+    <origin xyz="0 ${arm_length} ${rotor_z_offset}" rpy="0 0 0" />
+    <xacro:insert_block name="rotor_inertia" />
   </xacro:vertical_rotor>
   <!--
@@ -79,6 +79,6 @@
     direction="cw" parent="${namespace}/base_link" mass="${rotor_mass}"
     radius="${rotor_radius}" id="2" color="Blue">
-    <origin xyz="-${arm_length} 0 ${rotor_z_offset}" rpy="0 0 0"/>
-    <xacro:insert_block name="rotor_inertia"/>
+    <origin xyz="-${arm_length} 0 ${rotor_z_offset}" rpy="0 0 0" />
+    <xacro:insert_block name="rotor_inertia" />
   </xacro:vertical_rotor>
   <!--
@@ -88,6 +88,6 @@
     direction="ccw" parent="${namespace}/base_link" mass="${rotor_mass}"
     radius="${rotor_radius}" id="3" color="Blue">
-    <origin xyz="0 -${arm_length} ${rotor_z_offset}" rpy="0 0 0"/>
-    <xacro:insert_block name="rotor_inertia"/>
+    <origin xyz="0 -${arm_length} ${rotor_z_offset}" rpy="0 0 0" />
+    <xacro:insert_block name="rotor_inertia" />
   </xacro:vertical_rotor>
 </robot>

File: mav_description/urdf/multirotor_base.urdf.xacro (robot description, xacro)
@@ -21,5 +21,5 @@
     <inertia ixx="${(1.0/12.0) * mass * (y*y + z*z)}" ixy="0.0" ixz="0.0"
              iyy="${(1.0/12.0) * mass * (x*x + z*z)}" iyz="0.0"
-             izz="${(1.0/12.0) * mass * (x*x + y*y)}"/> <!-- [kg m^2] ... -->
+             izz="${(1.0/12.0) * mass * (x*x + y*y)}" /> <!-- [kg m^2] ... -->
   </xacro:macro>
   <!--
@@ -28,7 +28,7 @@
   <xacro:macro name="box_inertial" params="x y z mass *origin">
     <inertial>
-      <mass value="${mass}"/>
-      <xacro:insert_block name="origin"/>
-      <xacro:box_inertia x="${x}" y="${y}" z="${z}" mass="${mass}"/>
+      <mass value="${mass}" />
+      <xacro:insert_block name="origin" />
+      <xacro:box_inertia x="${x}" y="${y}" z="${z}" mass="${mass}" />
     </inertial>
   </xacro:macro>
@@ -42,25 +42,25 @@
     <link name="${robot_namespace}/base_link_inertia">
       <inertial>
-        <mass value="${mass}"/> <!-- [kg] -->
-        <origin xyz="0 0 0"/>
-        <xacro:insert_block name="inertia"/>
+        <mass value="${mass}" /> <!-- [kg] -->
+        <origin xyz="0 0 0" />
+        <xacro:insert_block name="inertia" />
       </inertial>
       <visual>
-        <origin xyz="0 0 0" rpy="0 0 0"/>
+        <origin xyz="0 0 0" rpy="0 0 0" />
         <geometry>
-          <mesh filename="${mesh_file}" scale="1 1 1"/>
+          <mesh filename="${mesh_file}" scale="1 1 1" />
         </geometry>
       </visual>
       <collision>
-        <origin xyz="0 0 0" rpy="0 0 0"/>
+        <origin xyz="0 0 0" rpy="0 0 0" />
         <geometry>
-          <box size="${length} ${width} ${height}"/> <!-- [m] [m] [m] -->
+          <box size="${length} ${width} ${height}" /> <!-- [m] [m] [m] -->
         </geometry>
       </collision>
     </link>
     <joint name="${robot_namespace}/base_joint" type="fixed">
-      <origin xyz="0 0 0" rpy="0 0 0"/>
-      <parent link="${robot_namespace}/base_link"/>
-      <child link="${robot_namespace}/base_link_inertia"/>
+      <origin xyz="0 0 0" rpy="0 0 0" />
+      <parent link="${robot_namespace}/base_link" />
+      <child link="${robot_namespace}/base_link_inertia" />
     </joint>
   </xacro:macro>
@@ -72,24 +72,24 @@
     <link name="${robot_namespace}/rotor_${id}">
       <inertial>
-        <mass value="${mass}"/> <!-- [kg] -->
-        <xacro:insert_block name="inertia"/>
+        <mass value="${mass}" /> <!-- [kg] -->
+        <xacro:insert_block name="inertia" />
       </inertial>
       <visual>
         <geometry>
           <mesh filename="file://$(find mav_description)/meshes/propeller_${direction}.dae"
-            scale="${radius} ${radius} ${radius}"/> <!-- [m] [m] [m] -->
+            scale="${radius} ${radius} ${radius}" /> <!-- [m] [m] [m] -->
         </geometry>
       </visual>
       <collision>
         <geometry>
-          <cylinder length="0.005" radius="${radius}"/> <!-- [m] -->
+          <cylinder length="0.005" radius="${radius}" /> <!-- [m] -->
         </geometry>
       </collision>
     </link>
     <joint name="${robot_namespace}/rotor_${id}_joint" type="continuous">
-      <xacro:insert_block name="origin"/>
-      <axis xyz="0 0 1"/>
-      <parent link="${parent}"/>
-      <child link="${robot_namespace}/rotor_${id}"/>
+      <xacro:insert_block name="origin" />
+      <axis xyz="0 0 1" />
+      <parent link="${parent}" />
+      <child link="${robot_namespace}/rotor_${id}" />
     </joint>
     <gazebo>

Commit message: Added multirotor_controller plugin boiler plate code

File: mav_description/urdf/hummingbird.urdf.xacro (robot description, xacro)
@@ -15,6 +15,14 @@
 <robot name="hummingbird" xmlns:xacro="http://ros.org/wiki/xacro">
   <!--
-    Include the hummingbird base xacro
+    Include the multirotor generic components
+  -->
+  <xacro:include filename="$(find mav_description)/urdf/mav_generic_components.xacro" />
+  <!--
+    Instantiate the hummingbird mechanics
   -->
   <xacro:include filename="$(find mav_description)/urdf/hummingbird_base.urdf.xacro" />
+  <!--
+    Instantiate the corresponding controller
+  -->
+  <xacro:multirotor_controller robot_namespace="$(arg namespace)" />
 </robot>

File: mav_description/urdf/mav_generic_components.xacro (robot description, xacro)
@@ -14,3 +14,18 @@
 -->
 <robot xmlns:xacro="http://ros.org/wiki/xacro">
+  <!--
+    Macro for the multirotor's controller interface
+  -->
+  <xacro:macro name="multirotor_controller" params="robot_namespace">
+    <gazebo>
+      <plugin name="${robot_namespace}_multirotor_controller"
+        filename="libgazebo_ros_multirotor_controller.so">
+        <!-- -->
+        <ros>
+          <namespace>${robot_namespace}</namespace>
+        </ros>
+        <link_name>${robot_namespace}/base_link</link_name>
+      </plugin>
+    </gazebo>
+  </xacro:macro>
 </robot>

File: mav_description/urdf/multirotor_base.urdf.xacro (robot description, xacro)
@@ -70,6 +70,10 @@
         <ros>
           <namespace>${robot_namespace}</namespace>
+          <remapping>joint_states:=joint_states</remapping>
         </ros>
         <link_name>${robot_namespace}/base_link</link_name>
+        <!-- -->
+        <publish_states>true</publish_states>
+        <update_rate>100.0</update_rate>
       </plugin>
     </gazebo>

Commit message: Changes to add imu_sensor's link

File: mav_description/urdf/hummingbird.urdf.xacro (robot description, xacro)
@@ -25,4 +25,14 @@
     Instantiate the corresponding controller
   -->
-  <xacro:multirotor_controller robot_namespace="$(arg namespace)" />
+  <xacro:multirotor_controller robot_namespace="${namespace}" />
+  <!--
+    Instantiate the imu sensor
+  -->
+  <xacro:imu_sensor robot_namespace="${namespace}" mass="0.00001"
+    parent="${namespace}/base_link">
+    <inertia ixx="0.00001" ixy="0.0" ixz="0.0"
+             iyy="0.00001" iyz="0.0"
+             izz="0.00001" /> <!-- [kg m^2] ... -->
+    <origin xyz="0 0 0" rpy="0 0 0" />
+  </xacro:imu_sensor>
 </robot>

File: mav_description/urdf/mav_generic_components.xacro (robot description, xacro)
@@ -33,3 +33,21 @@
     </gazebo>
   </xacro:macro>
+  <!--
+    Macro for the multirotor's IMU sensor
+  -->
+  <xacro:macro name="imu_sensor"
+    params="robot_namespace parent mass *inertia *origin">
+    <link name="${robot_namespace}/imu_link">
+      <inertial>
+        <mass value="${mass}" /> <!-- [kg] -->
+        <xacro:insert_block name="inertia" />
+      </inertial>
+      <!-- no visual and collision entries -->
+    </link>
+    <joint name="${robot_namespace}/imu_joint" type="fixed">
+      <xacro:insert_block name="origin" />
+      <parent link="${parent}" />
+      <child link="${robot_namespace}/imu_link" />
+    </joint>
+  </xacro:macro>
 </robot>

File: mav_description/urdf/multirotor_base.urdf.xacro (robot description, xacro)
@@ -85,5 +85,5 @@
   <xacro:macro name="vertical_rotor"
     params="robot_namespace suffix direction parent mass radius id color *origin *inertia">
-    <link name="${robot_namespace}/rotor_${id}">
+    <link name="${robot_namespace}/rotor_${id}_link">
       <inertial>
         <mass value="${mass}" /> <!-- [kg] -->
@@ -106,5 +106,5 @@
       <axis xyz="0 0 1" />
       <parent link="${parent}" />
-      <child link="${robot_namespace}/rotor_${id}" />
+      <child link="${robot_namespace}/rotor_${id}_link" />
     </joint>
     <gazebo>
@@ -119,5 +119,5 @@
         <!-- -->
         <joint_name>${robot_namespace}/rotor_${id}_joint</joint_name>
-        <link_name>${robot_namespace}/rotor_${id}</link_name>
+        <link_name>${robot_namespace}/rotor_${id}_link</link_name>
         <rotation_direction>${direction}</rotation_direction>
         <control_type>angular_speed</control_type>
@@ -127,5 +127,5 @@
       </plugin>
     </gazebo>
-    <gazebo reference="${robot_namespace}/rotor_${id}">
+    <gazebo reference="${robot_namespace}/rotor_${id}_link">
       <material>Gazebo/${color}</material>
     </gazebo>

Commit message: Changes for imu.urdf.xacro

File: mav_description/urdf/hummingbird.urdf.xacro (robot description, xacro)
@@ -19,4 +19,8 @@
   <xacro:include filename="$(find mav_description)/urdf/mav_generic_components.xacro" />
   <!--
+    Include the imu sensor
+  -->
+  <xacro:include filename="$(find mav_description)/urdf/imu.urdf.xacro" />
+  <!--
     Instantiate the hummingbird mechanics
   -->
@@ -29,9 +33,6 @@
     Instantiate the imu sensor
   -->
-  <xacro:imu_sensor robot_namespace="${namespace}" mass="0.00001"
+  <xacro:imu_sensor robot_namespace="${namespace}" color="Black"
     parent="${namespace}/base_link">
-    <inertia ixx="0.00001" ixy="0.0" ixz="0.0"
-             iyy="0.00001" iyz="0.0"
-             izz="0.00001" /> <!-- [kg m^2] ... -->
     <origin xyz="0 0 0" rpy="0 0 0" />
   </xacro:imu_sensor>

File: mav_description/urdf/mav_generic_components.xacro (robot description, xacro)
@@ -33,21 +33,3 @@
     </gazebo>
   </xacro:macro>
-  <!--
-    Macro for the multirotor's IMU sensor
-  -->
-  <xacro:macro name="imu_sensor"
-    params="robot_namespace parent mass *inertia *origin">
-    <link name="${robot_namespace}/imu_link">
-      <inertial>
-        <mass value="${mass}" /> <!-- [kg] -->
-        <xacro:insert_block name="inertia" />
-      </inertial>
-      <!-- no visual and collision entries -->
-    </link>
-    <joint name="${robot_namespace}/imu_joint" type="fixed">
-      <xacro:insert_block name="origin" />
-      <parent link="${parent}" />
-      <child link="${robot_namespace}/imu_link" />
-    </joint>
-  </xacro:macro>
 </robot>

Commit message: Changes for p3d interface

File: mav_description/urdf/hummingbird.urdf.xacro (robot description, xacro)
@@ -27,7 +27,11 @@
   <xacro:include filename="$(find mav_description)/urdf/hummingbird_base.urdf.xacro" />
   <!--
-    Instantiate the corresponding controller
+    Instantiate the hummingbird controller
   -->
   <xacro:multirotor_controller robot_namespace="${namespace}" />
+  <!--
+    Instantiate the gt p3d interface
+  -->
+  <xacro:gt_p3d robot_namespace="${namespace}" />
   <!--
     Instantiate the imu sensor

File: mav_description/urdf/mav_generic_components.xacro (robot description, xacro)
@@ -23,13 +23,44 @@
         <!-- -->
         <ros>
+          <!-- Add a namespace -->
           <namespace>${robot_namespace}</namespace>
+          <!-- Remap the actuator input topic -->
           <remapping>actuators_input:=command/motor_speed</remapping>
         </ros>
-        <!-- -->
+        <!-- Name of the link within this model whose actuators will be commanded -->
         <link_name>${robot_namespace}/base_link</link_name>
-        <!-- -->
+        <!-- Update rate in Hz, defaults to 0.0, which means as fast as possible -->
         <update_rate>0.0</update_rate>
       </plugin>
     </gazebo>
   </xacro:macro>
+  <!--
+    Macro for the multirotor's ground truth 3d position
+  -->
+  <xacro:macro name="gt_p3d" params="robot_namespace">
+    <gazebo>
+      <plugin name="${robot_namespace}_gt_p3d"
+          filename="libgazebo_ros_p3d.so">
+          <!-- -->
+          <ros>
+            <!-- Add a namespace -->
+            <namespace>${robot_namespace}</namespace>
+            <!-- Remap the odom topic -->
+            <remapping>odom:=odom</remapping>
+          </ros>
+          <!-- Name of the link within this model whose pose will be published -->
+          <body_name>${robot_namespace}/base_link</body_name>
+          <!-- Name of another link within this model to use as a reference frame -->
+          <frame_name>world</frame_name>
+          <!-- Update rate in Hz, defaults to 0.0, which means as fast as possible -->
+          <update_rate>0.0</update_rate>
+          <!-- Translation offset to be added to the pose. -->
+          <xyz_offset>0.0 0.0 0.0</xyz_offset>
+          <!-- Rotation offset to be added to the pose, in Euler angles. -->
+          <rpy_offset>0.0 0.0 0.0</rpy_offset>
+          <!-- Standard deviation of the noise to be added to the reported velocities. -->
+          <gaussian_noise>1.0e-2</gaussian_noise>
+      </plugin>
+    </gazebo>
+  </xacro:macro>
 </robot>

File: mav_description/urdf/multirotor_base.urdf.xacro (robot description, xacro)
@@ -69,11 +69,14 @@
         <!-- -->
         <ros>
+          <!-- Add a namespace -->
           <namespace>${robot_namespace}</namespace>
+          <!-- Remap the joint states topic -->
           <remapping>joint_states:=joint_states</remapping>
         </ros>
-        <!-- -->
+        <!-- Name of the link within this model whose actuators' joint state will be published -->
         <link_name>${robot_namespace}/base_link</link_name>
-        <!-- -->
+        <!-- Whether to publish the joint states -->
         <publish_states>true</publish_states>
+        <!-- Update rate in Hz, defaults to 0.0, which means as fast as possible -->
         <update_rate>0.0</update_rate>
       </plugin>
@@ -113,15 +116,22 @@
         <!-- -->
         <ros>
+          <!-- Add a namespace -->
           <namespace>${robot_namespace}</namespace>
+          <!-- Remap the motor angular velocity topic -->
           <remapping>angular_velocity:=rotor_${id}/angular_velocity</remapping>
+          <!-- Remap the motor control input topic -->
           <remapping>control_input:=rotor_${id}/control_input</remapping>
         </ros>
-        <!-- -->
+        <!-- Name of the motor joint within this model -->
         <joint_name>${robot_namespace}/rotor_${id}_joint</joint_name>
+        <!-- Name of the motor link within this model -->
         <link_name>${robot_namespace}/rotor_${id}_link</link_name>
+        <!-- motor rotation direction -->
         <rotation_direction>${direction}</rotation_direction>
+        <!-- motor control input type -->
         <control_type>angular_speed</control_type>
-        <!-- -->
+        <!-- Whether to publish the angular velocities -->
         <publish_velocity>true</publish_velocity>
+        <!-- Update rate in Hz, defaults to 0.0, which means as fast as possible -->
         <update_rate>0.0</update_rate>
       </plugin>
