Commit message: Minor code refactor

File: mav_description/urdf/hummingbird.urdf.xacro (robot description, xacro)
@@ -15,4 +15,8 @@
 <robot name="hummingbird" xmlns:xacro="http://ros.org/wiki/xacro">
   <!--
+    Arguments for the Asctec Hummingbird
+  -->
+  <xacro:arg name="namespace" default="hummingbird" />
+  <!--
     Include the multirotor generic components
   -->
@@ -29,14 +33,14 @@
     Instantiate the hummingbird controller
   -->
-  <xacro:multirotor_controller robot_namespace="${namespace}" />
+  <xacro:multirotor_controller robot_namespace="$(arg namespace)" />
   <!--
     Instantiate the gt p3d interface
   -->
-  <xacro:gt_p3d robot_namespace="${namespace}" />
+  <xacro:gt_p3d robot_namespace="$(arg namespace)" />
   <!--
     Instantiate the imu sensor
   -->
-  <xacro:imu_sensor robot_namespace="${namespace}" color="Black"
-    parent="${namespace}/base_link">
+  <xacro:imu_sensor robot_namespace="$(arg namespace)" color="Black"
+    parent="$(arg namespace)/base_link">
     <origin xyz="0 0 0" rpy="0 0 0" />
   </xacro:imu_sensor>

File: mav_description/urdf/hummingbird_base.urdf.xacro (robot description, xacro)
@@ -18,5 +18,5 @@
     reference Novel Dynamic Inversion Architectur Design for Quadrocopter Control by Wang et al.
   -->
-  <xacro:property name="namespace" value="$(arg namespace)" />
+  <xacro:property name="mav_namespace" value="$(arg namespace)" />
   <xacro:property name="mav_mesh_file" value="file://$(find mav_description)/meshes/hummingbird.dae" />
   <xacro:property name="body_mass" value="0.68" /> <!-- [kg] -->
@@ -50,5 +50,5 @@
     Instantiate the multirotor_base macro
   -->
-  <xacro:multirotor_base robot_namespace="${namespace}" mass="${body_mass}"
+  <xacro:multirotor_base robot_namespace="${mav_namespace}" mass="${body_mass}"
     length="${body_length}" width="${body_width}" height="${body_height}"
     mesh_file="${mav_mesh_file}">
@@ -58,6 +58,6 @@
     Instantiate the front vertical_rotor macro
   -->
-  <xacro:vertical_rotor robot_namespace="${namespace}" suffix="front"
-    direction="cw" parent="${namespace}/base_link" mass="${rotor_mass}"
+  <xacro:vertical_rotor robot_namespace="${mav_namespace}" suffix="front"
+    direction="cw" parent="${mav_namespace}/base_link" mass="${rotor_mass}"
     radius="${rotor_radius}" id="0" color="Red">
     <origin xyz="${arm_length} 0 ${rotor_z_offset}" rpy="0 0 0" />
@@ -67,6 +67,6 @@
     Instantiate the left vertical_rotor macro
   -->
-  <xacro:vertical_rotor robot_namespace="${namespace}" suffix="left"
-    direction="ccw" parent="${namespace}/base_link" mass="${rotor_mass}"
+  <xacro:vertical_rotor robot_namespace="${mav_namespace}" suffix="left"
+    direction="ccw" parent="${mav_namespace}/base_link" mass="${rotor_mass}"
     radius="${rotor_radius}" id="1" color="Blue">
     <origin xyz="0 ${arm_length} ${rotor_z_offset}" rpy="0 0 0" />
@@ -76,6 +76,6 @@
     Instantiate the back vertical_rotor macro
   -->
-  <xacro:vertical_rotor robot_namespace="${namespace}" suffix="back"
-    direction="cw" parent="${namespace}/base_link" mass="${rotor_mass}"
+  <xacro:vertical_rotor robot_namespace="${mav_namespace}" suffix="back"
+    direction="cw" parent="${mav_namespace}/base_link" mass="${rotor_mass}"
     radius="${rotor_radius}" id="2" color="Blue">
     <origin xyz="-${arm_length} 0 ${rotor_z_offset}" rpy="0 0 0" />
@@ -85,6 +85,6 @@
     Instantiate the right vertical_rotor macro
   -->
-  <xacro:vertical_rotor robot_namespace="${namespace}" suffix="right"
-    direction="ccw" parent="${namespace}/base_link" mass="${rotor_mass}"
+  <xacro:vertical_rotor robot_namespace="${mav_namespace}" suffix="right"
+    direction="ccw" parent="${mav_namespace}/base_link" mass="${rotor_mass}"
     radius="${rotor_radius}" id="3" color="Blue">
     <origin xyz="0 -${arm_length} ${rotor_z_offset}" rpy="0 0 0" />

File: mav_description/urdf/imu.urdf.xacro (robot description, xacro)
@@ -61,14 +61,16 @@
       <material>Gazebo/${color}</material>
       <sensor name="imu_sensor" type="imu">
+        <!-- Ensure sensor is always active -->
+        <always_on>true</always_on>
+        <!-- Update rate in Hz, defaults to 0.0, which means as fast as possible -->
+        <update_rate>100</update_rate>
         <!-- -->
-        <always_on>true</always_on>
-        <update_rate>100</update_rate>
-        <!-- IMU Noise -->
         <imu>
+          <!-- Angular velocity noise model [rad/s] -->
           <angular_velocity>
             <x>
               <noise type="gaussian">
                 <mean>0.0</mean>
-                <stddev>2e-4</stddev>
+                <stddev>2.0e-4</stddev>
               </noise>
             </x>
@@ -76,5 +78,5 @@
               <noise type="gaussian">
                 <mean>0.0</mean>
-                <stddev>2e-4</stddev>
+                <stddev>2.0e-4</stddev>
               </noise>
             </y>
@@ -82,8 +84,9 @@
               <noise type="gaussian">
                 <mean>0.0</mean>
-                <stddev>2e-4</stddev>
+                <stddev>2.0e-4</stddev>
               </noise>
             </z>
           </angular_velocity>
+          <!-- Linear acceleration noise model [m/s^2] -->
           <linear_acceleration>
             <x>
@@ -111,8 +114,10 @@
           <!-- -->
           <ros>
-            <namespace>${robot_namespace}/imu</namespace>
-            <remapping>~/out:=data</remapping>
+            <!-- Add a namespace -->
+            <namespace>${robot_namespace}</namespace>
+            <!-- Remap the imu topic -->
+            <remapping>~/out:=imu</remapping>
           </ros>
-          <!-- -->
+          <!-- To comply with REP 145 (world as orientation reference) -->
           <initial_orientation_as_reference>false</initial_orientation_as_reference>
         </plugin>
